File: knobbybox.kicad_sch (KiCad schematic)
At the start: 37 parts, among them J1 USB_C_Receptacle_USB2.0_14P, J2 SWD, U1 RP2354A, U2 AP2112K-3.3, Y1 Crystal

Commit message: micro layout
Parts:
- RESET1, USBDEV1: footprint USB-C-Power-tester:SW_Push_1P1T_NO_CK_KMR2 -> Button_Switch_SMD:SW_Push_1P1T_NO_CK_KSC6xxG
Changed lines of the file:
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@@
 			)
 		)
-		(property "Footprint" "USB-C-Power-tester:SW_Push_1P1T_NO_CK_KMR2"
+		(property "Footprint" "Button_Switch_SMD:SW_Push_1P1T_NO_CK_KSC6xxG"
 			(at 161.29 91.44 0)
 			(hide yes)
@@
 			)
 		)
-		(property "Footprint" "USB-C-Power-tester:SW_Push_1P1T_NO_CK_KMR2"
+		(property "Footprint" "Button_Switch_SMD:SW_Push_1P1T_NO_CK_KSC6xxG"
 			(at 161.29 73.66 0)
 			(hide yes)
