File: knobbybox.kicad_pcb (KiCad board)
At the start: 2 copper layers, 103 x 60 mm, 35 parts, among them J1 USB_C_Receptacle_USB2.0_14P, J2 SWD, U1 RP2354A, U2 AP2112K-3.3, Y1 Crystal

Commit message: micro layout
Parts:
- added RESET1: SW_Push, Button_Switch_SMD:SW_Push_1P1T_NO_CK_KSC6xxG, F.Cu at (22.6, -13.1)
- added USBDEV1: SW_Push, Button_Switch_SMD:SW_Push_1P1T_NO_CK_KSC6xxG, F.Cu at (22.6, -5.29)
- moved J2 51.9 mm to (41.3, 20.3), turned to 180 degrees
- moved R50 39.2 mm to (26.9, 25.3), turned to 180 degrees
- moved R51 38.7 mm to (26.9, 26.4)
- moved R52 38.1 mm to (26.9, 27.5)
- moved C25 37.5 mm to (39.6, 24.6)
- moved C29 37.2 mm to (39.6, 26.0), turned to 180 degrees
- moved R53 35.2 mm to (26.9, 24.2), turned to 180 degrees
- moved R54 35.1 mm to (23.5, 6.50)
- moved C27 33.2 mm to (33.4, 29.7), turned to 90 degrees
- moved C38 32.3 mm to (31.1, 29.7), turned to 90 degrees
- moved U2 28.6 mm to (26.1, 18.6)
- moved C39 28.4 mm to (37.9, 19.2), turned to -90 degrees
- moved C28 27.0 mm to (33.5, 19.2), turned to -90 degrees
- moved C40 25.0 mm to (29.5, 25.8), turned to 90 degrees
- moved C26 24.8 mm to (29.7, 18.4), turned to 180 degrees
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Routing:
- net /VBUS: track 0.00 -> 17.8 mm
- net +1V1: track 7.83 -> 20.5 mm, vias 2 -> 4
- net +3V3: track 17.4 -> 29.5 mm, vias 3 -> 7
- net /SIO: track 0.00 -> 7.93 mm, vias 0 -> 1
- net /SWC: track 0.00 -> 5.81 mm
- net Net-(U1-USB_DP): track 0.00 -> 4.50 mm
- net Net-(U1-USB_DM): track 0.00 -> 4.04 mm
- net Net-(U1-VREG_AVDD): track 0.00 -> 3.45 mm
- net Net-(J1-CC1): track 0.00 -> 2.88 mm
- net /USB_DP: track 2.82 -> 5.61 mm
- net Net-(J1-CC2): track 0.00 -> 2.76 mm
- net /VREG_LX: track 0.00 -> 2.23 mm
- net /USB_DM: track 2.74 -> 4.93 mm
- net Net-(U1-XOUT): track 3.81 -> 5.22 mm
- net GND: track 9.79 -> 9.11 mm, vias 0 -> 20
- added copper zone on B.Cu, net +3V3

Commit message: bla
Parts:
- RESET1, USBDEV1: footprint Button_Switch_SMD:SW_Push_1P1T_NO_CK_KSC6xxG -> Button_Switch_SMD:SW_SPST_CK_RS282G05A3
- moved R29 39.7 mm to (27.1, 15.1), turned to 180 degrees
- moved USBDEV1 39.4 mm to (23.1, 34.1), turned to 180 degrees
- moved R54 32.0 mm to (20.1, 38.3)
- moved RESET1 30.3 mm to (33.8, 15.1), turned to 180 degrees
Connections:
- U1 pad 27: /ENC_2A -> /DIR_1D
- U1 pad 28: /ENC_2B -> /DIR_1A
- U1 pad 29: /ENC_2C -> /PUSH_1
- U1 pad 31: /ENC_2D -> /DIR_1B
- U1 pad 32: /PUSH_2 -> /DIR_1C
- U1 pad 4: /DIR_1A -> /ENC_2B
- U1 pad 5: /DIR_1B -> /ENC_2D
- U1 pad 7: /DIR_1C -> /PUSH_2
- U1 pad 8: /DIR_1D -> /ENC_2A
- U1 pad 9: /PUSH_1 -> /ENC_2C
Routing:
- net /ENC_2A: track 0.00 -> 38.3 mm
- net /ENC_2C: track 0.00 -> 36.3 mm
- net /PUSH_2: track 0.00 -> 21.7 mm
- net /ENC_2B: track 0.00 -> 20.6 mm
- net /ENC_2D: track 0.00 -> 18.7 mm
- net Net-(U1-RUN): track 0.00 -> 10.5 mm, vias 0 -> 2
- net Net-(U1-~{QSPI_SS}): track 0.00 -> 9.13 mm
- net unconnected-(U1-GPIO1-Pad3): track 0.00 -> 7.23 mm
- net unconnected-(U1-GPIO0-Pad2): track 0.00 -> 6.69 mm
- net Net-(R54-Pad1): track 0.00 -> 4.23 mm
- net Net-(R29-Pad1): track 0.00 -> 1.97 mm
- net GND: vias 20 -> 26
